Commit message: Update turtlebot3_waffle_pi.urdf.xacro
remove camera for better performance

File: ros_multi_tb3/urdf/turtlebot3_waffle_pi.urdf.xacro (robot description, xacro)
@@ -161,10 +161,10 @@
     </inertial>
   </link>
-  <joint name="camera_joint" type="fixed">
+  <!--<joint name="camera_joint" type="fixed">
     <origin xyz="0.073 -0.011 0.084" rpy="0 0 0"/>
     <parent link="base_link"/>
     <child link="camera_link"/>
-  </joint>
-  <link name="camera_link">
+  </joint>-->
+  <!--<link name="camera_link">
     <collision>
       <origin xyz="0.005 0.011 0.013" rpy="0 0 0"/>
@@ -173,16 +173,16 @@
       </geometry>
     </collision>
-  </link>
-  <joint name="camera_rgb_joint" type="fixed">
+  </link>-->
+ <!-- <joint name="camera_rgb_joint" type="fixed">
     <origin xyz="0.003 0.011 0.009" rpy="0 0 0"/>
     <parent link="camera_link"/>
     <child link="camera_rgb_frame"/>
   </joint>
-  <link name="camera_rgb_frame"/>
-  <joint name="camera_rgb_optical_joint" type="fixed">
+  <link name="camera_rgb_frame"/>-->
+  <!--<joint name="camera_rgb_optical_joint" type="fixed">
     <origin xyz="0 0 0" rpy="-1.57 0 -1.57"/>
     <parent link="camera_rgb_frame"/>
     <child link="camera_rgb_optical_frame"/>
   </joint>
-  <link name="camera_rgb_optical_frame"/>
+  <link name="camera_rgb_optical_frame"/> -->
 </robot>
